File: Elec/PCB/kicad_files/anavi-play-phat.kicad_pcb (KiCad board)
At the start: 2 copper layers, 77.6 x 30 mm, 13 parts, among them J2 USB_A_PLUG

Commit message: pcb
Parts:
- J2: moved to B.Cu
- turned J2 to 90 degrees
Routing:
- net (no net): track 135.9 -> 96.5 mm, vias 4 -> 2
- net +5V: track 0.46 -> 21.8 mm, vias 0 -> 1
- net Net-(RASP_CONN1-Pad5): track 29.4 -> 19.1 mm
- net Net-(RASP_CONN1-Pad3): track 21.2 -> 27.9 mm
- net GND: track 28.6 -> 29.6 mm
Other:
- board text added: "D+"
- board text added: "D-"
