File: Elec/PCB/kicad_files/anavi-play-phat.kicad_pcb (KiCad board)
At the start: 2 copper layers, 79.5 x 30 mm, 15 parts, among them J1 d+ d-, J2 5v gnd, J2 USB_A_PLUG

Commit message: IL EST ECRIT QUE SEUL LONK PEUT VAINCRE GANON
Connections:
- J2 pad 1: GND -> +5V
- J2 pad 4: +5V -> GND
Routing:
- net +5V: track 26.0 -> 19.7 mm
Changed lines of the file:
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@@
     (thickness 1.6)
     (drawings 20)
-    (tracks 101)
+    (tracks 99)
     (zones 0)
     (modules 15)
@@
   )
   (setup
-    (last_trace_width 0.5)
+    (last_trace_width 1)
     (user_trace_width 0.254)
     (user_trace_width 0.5)
@@
     (mod_text_size 1 1)
     (mod_text_width 0.15)
-    (pad_size 1.8 1.8)
-    (pad_drill 1.2)
+    (pad_size 1.9 8)
+    (pad_drill 0)
     (pad_to_mask_clearance 0)
     (aux_axis_origin 0 0)
@@
     (pad 3 connect rect (at -1.3 5.15 270) (size 2 7.5) (layers B.Cu B.Mask))
     (pad 4 connect rect (at -3.81 4.9 270) (size 1.9 8) (layers B.Cu B.Mask)
+      (net 2 GND))
+    (pad 1 connect rect (at 3.81 4.9 270) (size 1.9 8) (layers B.Cu B.Mask)
       (net 3 +5V))
-    (pad 1 connect rect (at 3.81 4.9 270) (size 1.9 8) (layers B.Cu B.Mask)
-      (net 2 GND))
   )
   (module boutton:boutton__6mx6m (layer B.Cu)
@@
       (rotate (xyz 0 0 90))
     )
-    (model /home/thibault/CIR4/KeyBox/Elec/PCB/libs/pins2*20.step
+    (model /home/thibault/CIR4/KeyBox/Elec/PCB/libs/pins2x20.step
       (offset (xyz 0 0 2.75))
       (scale (xyz 1 1 1))
@@
   (segment (start 187.4892 90.3732) (end 206.052987 90.3732) (width 1) (layer B.Cu) (net 1))
   (segment (start 176.8652 79.7492) (end 187.4892 90.3732) (width 1) (layer B.Cu) (net 1))
-  (segment (start 218.8932 94.4672) (end 213.8932 94.4672) (width 1) (layer B.Cu) (net 2))
-  (segment (start 213.8932 94.4672) (end 213.4316 94.4672) (width 1) (layer B.Cu) (net 2))
-  (segment (start 213.4316 94.4672) (end 211.7344 96.1644) (width 1) (layer B.Cu) (net 2))
-  (segment (start 203.001922 99.9744) (end 211.2264 91.749922) (width 1) (layer F.Cu) (net 3))
-  (segment (start 211.2264 91.749922) (end 211.2264 86.9188) (width 1) (layer F.Cu) (net 3))
-  (via (at 211.2264 86.9188) (size 1.8) (drill 1.2) (layers F.Cu B.Cu) (net 3))
-  (segment (start 218.8216 86.9188) (end 218.8932 86.8472) (width 1) (layer B.Cu) (net 3))
-  (segment (start 211.2264 86.9188) (end 218.8216 86.9188) (width 1) (layer B.Cu) (net 3))
+  (segment (start 218.8932 94.4672) (end 213.8932 94.4672) (width 1) (layer B.Cu) (net 3))
+  (segment (start 213.8932 94.4672) (end 213.4316 94.4672) (width 1) (layer B.Cu) (net 3))
+  (segment (start 213.4316 94.4672) (end 211.7344 96.1644) (width 1) (layer B.Cu) (net 3))
+  (via (at 211.582 96.52) (size 1.8) (drill 1.2) (layers F.Cu B.Cu) (net 3))
+  (segment (start 218.8216 86.9188) (end 218.8932 86.8472) (width 1) (layer B.Cu) (net 2))
+  (segment (start 211.2264 86.9188) (end 218.8216 86.9188) (width 1) (layer B.Cu) (net 2))
   (segment (start 156.5452 77.2092) (end 156.5402 77.1652) (width 0.5) (layer F.Cu) (net 3) (status 80000))
   (segment (start 156.5452 77.2092) (end 156.2422 77.2092) (width 0.5) (layer B.Cu) (net 3))
   (segment (start 156.5452 77.2092) (end 156.4327 77.2092) (width 0.5) (layer B.Cu) (net 3))
-  (segment (start 202.916322 99.8888) (end 201.6252 99.8888) (width 1) (layer F.Cu) (net 3))
-  (segment (start 203.001922 99.9744) (end 202.916322 99.8888) (width 1) (layer F.Cu) (net 3))
+  (segment (start 204.994 96.52) (end 211.582 96.52) (width 1) (layer F.Cu) (net 3))
+  (segment (start 201.6252 99.8888) (end 204.994 96.52) (width 1) (layer F.Cu) (net 3))
   (segment (start 169.2402 79.7052) (end 169.2452 79.7492) (width 0.5) (layer F.Cu) (net 4) (status 80000))
   (segment (start 168.381601 80.612799) (end 169.2452 79.7492) (width 1) (layer B.Cu) (net 4))
