File: Elec/PCB/kicad_files/anavi-play-phat.kicad_pcb (KiCad board)
At the start: 2 copper layers, 79.5 x 30 mm, 15 parts, among them J1 d+ d-, J2 5v gnd, J2 USB_A_PLUG

Commit message: Tout plein de modifs
Parts:
- J1: value d+ d- -> USB Data
- J2: value 5v gnd -> USB power
- moved J1 0.15 mm to (189.5, 102.3), turned to 180 degrees
Connections:
- net Net-(J1-Pad2) renamed D-
- J1 pad 1: Net-(J1-Pad1) -> D+
- J2 pad 1: GND -> +5V
- J2 pad 2: +5V -> GND
Routing:
- net D+: track 0.00 -> 43.2 mm, vias 0 -> 1
- net Net-(J1-Pad1): track 36.2 -> 0.00 mm
- net D-: track 33.1 -> 42.0 mm
Changed lines of the file:
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@@
     (thickness 1.6)
     (drawings 20)
-    (tracks 99)
+    (tracks 104)
     (zones 0)
     (modules 15)
@@
     (mod_text_size 1 1)
     (mod_text_width 0.15)
-    (pad_size 1.9 8)
+    (pad_size 2 7.5)
     (pad_drill 0)
     (pad_to_mask_clearance 0)
@@
   (net 30 "Net-(OK1-Pad2)")
   (net 31 "Net-(R1-Pad2)")
-  (net 32 "Net-(J1-Pad2)")
-  (net 33 "Net-(J1-Pad1)")
+  (net 32 D-)
+  (net 33 D+)
   (net_class Default "This is the default net class."
     (clearance 0.254)
@@
     (add_net +3V3)
     (add_net +5V)
+    (add_net D+)
+    (add_net D-)
     (add_net GND)
     (add_net "Net-(BCK1-Pad2)")
     (add_net "Net-(DWN1-Pad2)")
-    (add_net "Net-(J1-Pad1)")
-    (add_net "Net-(J1-Pad2)")
     (add_net "Net-(L1-Pad2)")
     (add_net "Net-(OK1-Pad2)")
@@
       (effects (font (size 1 1) (thickness 0.15)))
     )
-    (fp_text value "5v gnd" (at 0 -2.54 90) (layer F.SilkS)
+    (fp_text value "USB power" (at 0 -2.54 90) (layer F.SilkS)
       (effects (font (size 1 1) (thickness 0.15)))
     )
     (pad 2 thru_hole circle (at 1 0 90) (size 1.524 1.524) (drill 0.762) (layers *.Cu *.Mask)
+      (net 2 GND))
+    (pad 1 thru_hole circle (at -1 0 90) (size 1.524 1.524) (drill 0.762) (layers *.Cu *.Mask)
       (net 3 +5V))
-    (pad 1 thru_hole circle (at -1 0 90) (size 1.524 1.524) (drill 0.762) (layers *.Cu *.Mask)
-      (net 2 GND))
   )
   (module "w_conn_misc:header 2m spaced" (layer F.Cu)
-    (at 189.5508 102.4128)
+    (at 189.5348 102.2604 180)
     (fp_text reference J1 (at 0 2.54) (layer F.SilkS) hide
       (effects (font (size 1 1) (thickness 0.15)))
     )
-    (fp_text value "d+ d-" (at 0 -2.54) (layer F.SilkS)
-      (effects (font (size 1 1) (thickness 0.15)))
-    )
-    (pad 2 thru_hole circle (at 1 0) (size 1.524 1.524) (drill 0.762) (layers *.Cu *.Mask)
-      (net 32 "Net-(J1-Pad2)"))
-    (pad 1 thru_hole circle (at -1 0) (size 1.524 1.524) (drill 0.762) (layers *.Cu *.Mask)
-      (net 33 "Net-(J1-Pad1)"))
+    (fp_text value "USB Data" (at -0.1016 2.3368) (layer F.SilkS)
+      (effects (font (size 1 1) (thickness 0.15)))
+    )
+    (pad 2 thru_hole circle (at 1 0 180) (size 1.524 1.524) (drill 0.762) (layers *.Cu *.Mask)
+      (net 32 D-))
+    (pad 1 thru_hole circle (at -1 0 180) (size 1.524 1.524) (drill 0.762) (layers *.Cu *.Mask)
+      (net 33 D+))
   )
   (module i2c_screen:i2c_screen (layer B.Cu)
@@
       (effects (font (size 1 1) (thickness 0.15)) (justify mirror))
     )
-    (pad 2 connect rect (at 1.3 5.15 270) (size 2 7.5) (layers B.Cu B.Mask))
-    (pad 3 connect rect (at -1.3 5.15 270) (size 2 7.5) (layers B.Cu B.Mask))
+    (pad "" connect rect (at 1.3 5.15 270) (size 2 7.5) (layers B.Cu B.Mask)
+      (net 32 D-))
+    (pad "" connect rect (at -1.3 5.15 270) (size 2 7.5) (layers B.Cu B.Mask)
+      (net 33 D+))
     (pad 4 connect rect (at -3.81 4.9 270) (size 1.9 8) (layers B.Cu B.Mask)
       (net 2 GND))
@@
   (segment (start 187.4892 90.3732) (end 206.052987 90.3732) (width 1) (layer B.Cu) (net 1))
   (segment (start 176.8652 79.7492) (end 187.4892 90.3732) (width 1) (layer B.Cu) (net 1))
+  (segment (start 218.8216 86.9188) (end 218.8932 86.8472) (width 1) (layer B.Cu) (net 2))
+  (segment (start 211.2264 86.9188) (end 218.8216 86.9188) (width 1) (layer B.Cu) (net 2))
   (segment (start 218.8932 94.4672) (end 213.8932 94.4672) (width 1) (layer B.Cu) (net 3))
   (segment (start 213.8932 94.4672) (end 213.4316 94.4672) (width 1) (layer B.Cu) (net 3))
   (segment (start 213.4316 94.4672) (end 211.7344 96.1644) (width 1) (layer B.Cu) (net 3))
   (via (at 211.582 96.52) (size 1.8) (drill 1.2) (layers F.Cu B.Cu) (net 3))
-  (segment (start 218.8216 86.9188) (end 218.8932 86.8472) (width 1) (layer B.Cu) (net 2))
-  (segment (start 211.2264 86.9188) (end 218.8216 86.9188) (width 1) (layer B.Cu) (net 2))
   (segment (start 156.5452 77.2092) (end 156.5402 77.1652) (width 0.5) (layer F.Cu) (net 3) (status 80000))
   (segment (start 156.5452 77.2092) (end 156.2422 77.2092) (width 0.5) (layer B.Cu) (net 3))
@@
   (segment (start 161.657318 81.9912) (end 163.035719 80.612799) (width 0.254) (layer B.Cu) (net 31))
   (segment (start 160.8836 81.9912) (end 161.657318 81.9912) (width 0.254) (layer B.Cu) (net 31))
-  (segment (start 192.523998 100.446001) (end 192.690799 100.2792) (width 1) (layer B.Cu) (net 32))
-  (segment (start 190.6016 101.346) (end 191.501599 100.446001) (width 1) (layer B.Cu) (net 32))
-  (segment (start 191.501599 100.446001) (end 192.523998 100.446001) (width 1) (layer B.Cu) (net 32))
-  (segment (start 192.690799 100.2792) (end 195.2752 100.2792) (width 1) (layer B.Cu) (net 32))
-  (segment (start 195.2752 100.2792) (end 198.4248 97.1296) (width 1) (layer B.Cu) (net 32))
-  (segment (start 198.4248 97.1296) (end 208.8388 97.1296) (width 1) (layer B.Cu) (net 32))
-  (segment (start 213.8932 91.9572) (end 218.6432 91.9572) (width 1) (layer B.Cu) (net 32))
-  (segment (start 208.8388 97.0116) (end 213.8932 91.9572) (width 1) (layer B.Cu) (net 32))
-  (segment (start 208.8388 97.1296) (end 208.8388 97.0116) (width 1) (layer B.Cu) (net 32))
-  (segment (start 190.6016 101.346) (end 190.6016 102.4492) (width 1) (layer B.Cu) (net 32))
-  (segment (start 213.8932 89.3572) (end 207.9496 95.3008) (width 1) (layer B.Cu) (net 33))
-  (segment (start 191.082799 98.832801) (end 188.6204 101.2952) (width 1) (layer B.Cu) (net 33))
-  (segment (start 194.071921 98.832801) (end 191.082799 98.832801) (width 1) (layer B.Cu) (net 33))
-  (segment (start 218.6432 89.3572) (end 213.8932 89.3572) (width 1) (layer B.Cu) (net 33))
-  (segment (start 207.9496 95.3008) (end 197.603922 95.3008) (width 1) (layer B.Cu) (net 33))
-  (segment (start 197.603922 95.3008) (end 194.071921 98.832801) (width 1) (layer B.Cu) (net 33))
-  (segment (start 188.6204 102.3476) (end 188.5188 102.4492) (width 1) (layer B.Cu) (net 33))
-  (segment (start 188.6204 101.2952) (end 188.6204 102.3476) (width 1) (layer B.Cu) (net 33))
+  (segment (start 188.6204 102.3476) (end 188.5188 102.4492) (width 1) (layer B.Cu) (net 32))
+  (segment (start 216.828199 92.0588) (end 216.078199 91.3088) (width 0.8) (layer B.Cu) (net 32))
+  (segment (start 216.078199 91.3088) (end 213.507018 91.3088) (width 0.8) (layer B.Cu) (net 32))
+  (segment (start 222.4532 92.0588) (end 216.828199 92.0588) (width 0.8) (layer B.Cu) (net 32))
+  (segment (start 213.507018 91.3088) (end 208.050618 96.7652) (width 0.8) (layer B.Cu) (net 32))
+  (segment (start 208.050618 96.7652) (end 195.453782 96.7652) (width 0.8) (layer B.Cu) (net 32))
+  (segment (start 195.453782 96.7652) (end 193.726582 95.038) (width 0.8) (layer B.Cu) (net 32))
+  (segment (start 193.726582 95.038) (end 192.963018 95.038) (width 0.8) (layer B.Cu) (net 32))
+  (segment (start 192.963018 95.038) (end 189.965818 98.0352) (width 0.8) (layer B.Cu) (net 32))
+  (segment (start 188.5348 99.466218) (end 188.5348 102.2604) (width 1) (layer B.Cu) (net 32))
+  (segment (start 189.965818 98.0352) (end 188.5348 99.466218) (width 1) (layer B.Cu) (net 32))
+  (segment (start 216.828199 89.4588) (end 216.078199 90.2088) (width 0.8) (layer B.Cu) (net 33))
+  (segment (start 222.4532 89.4588) (end 216.828199 89.4588) (width 0.8) (layer B.Cu) (net 33))
+  (segment (start 216.078199 90.2088) (end 213.051382 90.2088) (width 0.8) (layer B.Cu) (net 33))
+  (segment (start 213.051382 90.2088) (end 207.594982 95.6652) (width 0.8) (layer B.Cu) (net 33))
+  (segment (start 207.594982 95.6652) (end 195.909418 95.6652) (width 0.8) (layer B.Cu) (net 33))
+  (segment (start 195.909418 95.6652) (end 194.182218 93.938) (width 0.8) (layer B.Cu) (net 33))
+  (segment (start 194.182218 93.938) (end 192.507382 93.938) (width 0.8) (layer B.Cu) (net 33))
+  (segment (start 192.507382 93.938) (end 189.510182 96.9352) (width 0.8) (layer B.Cu) (net 33))
+  (segment (start 189.510182 96.9352) (end 189.510182 96.9352) (width 0.8) (layer B.Cu) (net 33))
+  (via (at 189.510182 96.9352) (size 0.85) (drill 0.4) (layers F.Cu B.Cu) (net 33))
+  (segment (start 190.5348 97.959818) (end 190.5348 102.2604) (width 1) (layer F.Cu) (net 33))
+  (segment (start 189.510182 96.9352) (end 190.5348 97.959818) (width 1) (layer F.Cu) (net 33))
   (zone (net 0) (net_name "") (layers F&B.Cu) (hatch edge 0.508)
     (connect_pads (clearance 0.508))
@@
     (polygon
       (pts
-        (xy 227.7364 96.4184) (xy 215.0364 96.4438) (xy 214.9348 84.8106) (xy 227.7364 84.7344)
+        (xy 227.7364 96.4184) (xy 224.4852 96.4438) (xy 224.3836 84.8106) (xy 227.7364 84.7344)
       )
     )
